File: Hardware/dd.kicad_pcb (KiCad board)
At the start: 2 copper layers, 40.6 x 109.2 mm, 67 parts, among them CON1 AVR-ISP-6, J1 , J2 , J3 Conn_02x05_Odd_Even, J4 , J5 Conn_01x08_Male, J6 , J7 Conn_01x02_Male, Q1 MMBT3904, Q2 MMBT3904, Q3 MMBT3904, Q4 MMBT3904, Q5 MMBT3904, Q6 MMBT3904, Q7 MMBT3904, Q8 MMBT3904, U1 ATMEGA328P-AU, U2 MCP23S17, U3 LM1117-5.0, U4 MCP6002-xSN, Y1 20MHz

Commit message: footprint changed
Parts:
- U2: footprint SMD_Packages:SOIC-28 -> Housings_SOIC:SOIC-28W_7.5x17.9mm_Pitch1.27mm
- moved C4 3.40 mm to (60.2, 110.1)
- moved U2 1.22 mm to (63.9, 123.7), turned to 180 degrees
Connections:
- J1 pad 5: Net-(J1-Pad5) -> (no net)
- J2 pad 4: Net-(J2-Pad4) -> (no net)
- J2 pad 8: Net-(J2-Pad8) -> (no net)
- J5 pad 6: Net-(J5-Pad6) -> (no net)
- U1 pad 19: Net-(U1-Pad19) -> (no net)
- U2 pad 19: Net-(U2-Pad19) -> (no net)
- U2 pad 20: Net-(U2-Pad20) -> (no net)
- U2 pad 7: Net-(U2-Pad7) -> (no net)
- U4 pad 2: Net-(U4-Pad2) -> Net-(U4-Pad1)
- U4 pad 3: Net-(U4-Pad3) -> Net-(R25-Pad1)
Routing:
- net Net-(R25-Pad1): track 8.25 -> 13.6 mm
- net Net-(J1-Pad3): track 7.72 -> 12.2 mm, vias 0 -> 1
- net GND: track 369.0 -> 372.4 mm, vias 3 -> 5
- net Net-(CON1-Pad3): track 42.8 -> 39.6 mm
- net Net-(CON1-Pad1): track 49.0 -> 46.3 mm
- net Net-(C3-Pad1): track 64.4 -> 61.8 mm
- net Net-(J2-Pad3): track 36.9 -> 39.2 mm
- net Net-(J2-Pad2): track 38.2 -> 40.1 mm
- net Net-(R5-Pad2): track 29.1 -> 30.9 mm
- net Net-(J2-Pad6): track 31.5 -> 33.2 mm
- net Net-(U1-Pad14): track 34.1 -> 32.7 mm
- net Net-(J2-Pad7): track 30.5 -> 31.9 mm
- net Net-(U4-Pad1): track 0.00 -> 1.27 mm
- net VCC: track 172.0 -> 170.8 mm, vias 7 -> 6
- net Net-(CON1-Pad4): track 59.8 -> 58.7 mm
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